File: WordClockNorwegian.kicad_pcb (KiCad board)
At the start: 2 copper layers, 280 x 280 mm, 171 parts, among them CON1 AVR-ISP-6, IC1 ATMEGA328P-A, J1 CONN_Barrel-2.1mm_RASM722X_CPL, J2 0R, J3 0R, P1 CONN_01X06, SW1 SW_PUSH, SW2 SW_PUSH, SW3 SW_PUSH, U1 APA102, U10 DS1307_CPL, U11 APA102, U12 APA102, U13 APA102, U14 APA102, U15 APA102, U16 APA102, U17 APA102, U18 APA102, U19 APA102, U2 APA102, U20 APA102, U21 APA102, U22 APA102, U23 APA102, U24 APA102, U25 APA102, U26 APA102, U27 APA102, U28 APA102, U29 APA102, U3 APA102, U30 APA102, U31 APA102, U32 APA102, U33 APA102, U34 APA102, U35 APA102, U36 APA102, U37 APA102, U38 APA102, U39 APA102, U4 APA102, U40 APA102, U41 APA102, U42 APA102, U43 APA102, U44 APA102, U45 APA102, U46 APA102, U47 APA102, U48 APA102, U49 APA102, U5 APA102, U50 APA102, U51 APA102, U52 APA102, U53 APA102, U54 APA102, U55 APA102, U56 APA102, U57 APA102, U58 APA102, U59 APA102, U6 APA102, U60 APA102, U61 APA102, U62 APA102, U63 APA102, U64 APA102, U65 APA102, U66 APA102, U67 APA102, U68 APA102, U69 APA102, U7 APA102, U70 APA102, U71 APA102, U8 APA102, U9 APA102

Commit message: add silk
Parts:
- added G***: LOGO, Custom:LOGO2, F.Cu at (162.0, 161.0)

Commit message: HUGE update plus add ignore for bak files
Parts:
- removed G***: LOGO, Custom:LOGO2
- removed REF** (x4): MountingHole_3mm, Mounting_Holes:MountingHole_3mm
- removed REG1: REG_Linear_LM1117IMP_CPL, Housings_SOT-23_SOT-143_TSOT-6:SOT-143_Handsoldering
- added J10: 0R, Resistors_SMD:R_0805_HandSoldering, F.Cu at (289.1, 213.5)
- added J11: 0R, Resistors_SMD:R_0805_HandSoldering, F.Cu at (286.0, 213.5)
- added J12: 0R, Resistors_SMD:R_0805_HandSoldering, F.Cu at (290.1, 258.5)
- added J13: 0R, Resistors_SMD:R_0805_HandSoldering, F.Cu at (287.0, 258.5)
- added J4: 0R, Resistors_SMD:R_0805_HandSoldering, F.Cu at (283.0, 176.0)
- added J5: 0R, Resistors_SMD:R_0805_HandSoldering, F.Cu at (280.0, 176.0)
- added J6: 0R, Resistors_SMD:R_0805_HandSoldering, F.Cu at (286.6, 101.0)
- added J7: 0R, Resistors_SMD:R_0805_HandSoldering, F.Cu at (283.6, 101.0)
- added J8: 0R, Resistors_SMD:R_0805_HandSoldering, F.Cu at (289.8, 136.0)
- added J9: 0R, Resistors_SMD:R_0805_HandSoldering, F.Cu at (287.2, 136.0)
- added P2: CONN_01X02, Footprints:DO-214, F.Cu at (289.0, 282.2)
- added U72: LM1085ISX-5.0, Footprints:TO-263, F.Cu at (129.4, 186.4)
- D1: value SS12 -> S3JB
- J1: footprint Connect:BARREL_JACK -> Footprints:RASM722X
- SW1, SW2, SW3: footprint Buttons_Switches_SMD:SW_SPST_FSMSM -> Footprints:B3U-3000P
- moved J1 68.6 mm to (28.8, 186.4), turned to 270 degrees
- moved C6 11.6 mm to (122.7, 191.0), turned to 180 degrees
- moved D2 9.86 mm to (107.5, 189.5), turned to 180 degrees
- moved SW3 8.10 mm to (300.0, 182.7), turned to 270 degrees
- moved C78 7.94 mm to (125.0, 179.0)
- moved C7 6.43 mm to (131.0, 179.0), turned to 180 degrees
- moved SW2 5.59 mm to (300.0, 167.5), turned to 270 degrees
- moved SW1 4.72 mm to (300.0, 141.0), turned to 270 degrees
Connections:
- U18 pad 1: Net-(U18-Pad1) -> Net-(J12-Pad2)
- U18 pad 2: Net-(U18-Pad2) -> Net-(J13-Pad2)
- U22 pad 5: Net-(U22-Pad5) -> Net-(J7-Pad1)
- U22 pad 6: Net-(U22-Pad6) -> Net-(J6-Pad1)
- U31 pad 1: Net-(U22-Pad6) -> Net-(J6-Pad2)
- U31 pad 2: Net-(U22-Pad5) -> Net-(J7-Pad2)
- U41 pad 5: Net-(U41-Pad5) -> Net-(J9-Pad1)
- U41 pad 6: Net-(U41-Pad6) -> Net-(J8-Pad1)
- U42 pad 5: Net-(U42-Pad5) -> Net-(J5-Pad1)
- U42 pad 6: Net-(U42-Pad6) -> Net-(J4-Pad1)
- U50 pad 1: Net-(U41-Pad6) -> Net-(J8-Pad2)
- U50 pad 2: Net-(U41-Pad5) -> Net-(J9-Pad2)
- U51 pad 1: Net-(U42-Pad6) -> Net-(J4-Pad2)
- U51 pad 2: Net-(U42-Pad5) -> Net-(J5-Pad2)
- U69 pad 5: /COUT6 -> Net-(J11-Pad1)
- U69 pad 6: /DOUT6 -> Net-(J10-Pad1)
- U8 pad 5: Net-(U18-Pad2) -> Net-(J13-Pad1)
- U8 pad 6: Net-(U18-Pad1) -> Net-(J12-Pad1)
Routing:
- net VCC: track 3584.9 -> 3950.1 mm
- net /COUT6: track 0.00 -> 279.9 mm
- net /DOUT6: track 0.00 -> 272.2 mm
- net Net-(J9-Pad2): track 0.00 -> 271.7 mm
- net Net-(J13-Pad2): track 0.00 -> 271.6 mm
- net Net-(J12-Pad2): track 0.00 -> 268.8 mm
- net Net-(J7-Pad2): track 0.00 -> 268.3 mm
- net Net-(J8-Pad2): track 0.00 -> 266.9 mm
- net Net-(J5-Pad2): track 0.00 -> 263.6 mm
- net Net-(J6-Pad2): track 0.00 -> 262.5 mm
- net Net-(J4-Pad2): track 0.00 -> 261.6 mm
- net Net-(IC1-Pad12): track 0.00 -> 213.6 mm, vias 0 -> 6
- net Net-(IC1-Pad24): track 0.00 -> 208.1 mm, vias 0 -> 1
- net (no net): track 0.00 -> 206.3 mm, vias 0 -> 2
- net Net-(IC1-Pad14): track 0.00 -> 195.8 mm, vias 0 -> 6
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- added copper zone on B.Cu, net GND
Other:
- board text added: "DOUT COUT"
- board text added: "FTDI 5v"
- board text added: "ISP"

Commit message: before sendoff, one more check to go
Parts:
- added BAT1: BAT_CR2032_MPD-BA2032SM_CPL, Footprints:BAT_TE_796136-1, F.Cu at (195.0, 151.0)
- added G***: LOGO, Custom:backplate_mask, B.Cu at (162.1, 160.0)
- added H1: M3_mount, Footprints:M3, F.Cu at (22.0, 21.0)
- added H2: M3_mount, Footprints:M3, F.Cu at (262.0, 71.0)
- added H3: M3_mount, Footprints:M3, F.Cu at (62.0, 251.0)
- added H4: M3_mount, Footprints:M3, F.Cu at (262.0, 251.0)
- added P3: CONN_01X01, Measurement_Points:Measurement_Point_Round-SMD-Pad_Small, F.Cu at (126.0, 154.0)
- added P4: CONN_01X01, Measurement_Points:Measurement_Point_Round-SMD-Pad_Small, F.Cu at (123.0, 154.0)
- P2: footprint Footprints:DO-214 -> Socket_Strips:Socket_Strip_Straight_1x02
- moved P2 12.5 mm to (289.5, 269.8)
Routing:
- net Net-(IC1-Pad23): track 0.00 -> 219.7 mm, vias 0 -> 2
- net (no net): track 206.3 -> 0.00 mm, vias 2 -> 0
- net Net-(BAT1-Pad1): track 0.00 -> 104.3 mm, vias 0 -> 2
- net Net-(IC1-Pad24): track 208.1 -> 226.6 mm, vias 1 -> 2
- net Net-(P2-Pad2): track 8.96 -> 22.4 mm
- net Net-(P2-Pad1): track 6.99 -> 19.7 mm
- net SCL: track 18.4 -> 25.3 mm
- net SDA: track 18.0 -> 22.0 mm
- net Net-(IC1-Pad13): track 186.3 -> 188.5 mm, vias 3 -> 4
- net Net-(U19-Pad2): track 38.7 -> 37.3 mm
- net Net-(IC1-Pad14): track 195.8 -> 194.6 mm
- net GND: track 541.5 -> 540.6 mm
Other:
- net class VCC: trace_width 0.55 -> 1
- board text added: "ATMEGA + DS1337"
- board text added: "POWER"
- board text added: "PS: Unlabled 0805 can be 0.1uF or nothing"
- board text added: "REV: 1."
- board text added: "designed by alexanderbrevig.com"
- board text added: "get yours at ordklokke.no"

Commit message: tweaks
Parts:
- added P5: CONN_01X01, Measurement_Points:Measurement_Point_Round-SMD-Pad_Small, F.Cu at (30.2, 43.0)
- added P6: CONN_01X01, Measurement_Points:Measurement_Point_Round-SMD-Pad_Small, F.Cu at (30.2, 45.2)
Routing:
- net Net-(IC1-Pad23): track 219.7 -> 223.1 mm
Changed lines of the file:
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@@
 (kicad_pcb (version 4) (host pcbnew "(2015-08-16 BZR 6097, Git b384c94)-product")
   (general
-    (links 501)
+    (links 503)
     (no_connects 0)
     (area 21.924999 20.924999 302.075001 301.075001)
     (thickness 1.6)
     (drawings 33)
-    (tracks 1596)
+    (tracks 1602)
     (zones 0)
-    (modules 186)
+    (modules 188)
     (nets 188)
   )
@@
     (visible_elements 7FFEFF7F)
     (pcbplotparams
-      (layerselection 0x00030_80000001)
-      (usegerberextensions false)
+      (layerselection 0x010f0_80000001)
+      (usegerberextensions true)
       (excludeedgelayer true)
       (linewidth 0.100000)
@@
       (outputformat 1)
       (mirror false)
-      (drillshape 1)
+      (drillshape 0)
       (scaleselection 1)
-      (outputdirectory ""))
+      (outputdirectory fab/))
   )
   (net 0 "")
@@
       (net 19 SCL))
   )
+  (module Measurement_Points:Measurement_Point_Round-SMD-Pad_Small (layer F.Cu)
+    (at 30.25 43)
+    (descr "Mesurement Point, Round, SMD Pad, DM 1.5mm,")
+    (tags "Mesurement Point, Round, SMD Pad, DM 1.5mm,")
+    (fp_text reference P5 (at 0 -1.75) (layer F.SilkS)
+      (effects (font (size 1 1) (thickness 0.15)))
+    )
+    (fp_text value CONN_01X01 (at 1.27 2.54) (layer F.Fab)
+      (effects (font (size 1 1) (thickness 0.15)))
+    )
+    (pad 1 smd circle (at 0 0) (size 1.524 1.524) (layers F.Cu F.Paste F.Mask)
+      (net 30 "Net-(IC1-Pad23)"))
+  )
+  (module Measurement_Points:Measurement_Point_Round-SMD-Pad_Small (layer F.Cu)
+    (at 30.25 45.25)
+    (descr "Mesurement Point, Round, SMD Pad, DM 1.5mm,")
+    (tags "Mesurement Point, Round, SMD Pad, DM 1.5mm,")
+    (fp_text reference P6 (at 0 1.75) (layer F.SilkS)
+      (effects (font (size 1 1) (thickness 0.15)))
+    )
+    (fp_text value CONN_01X01 (at 1.27 2.54) (layer F.Fab)
+      (effects (font (size 1 1) (thickness 0.15)))
+    )
+    (pad 1 smd circle (at 0 0) (size 1.524 1.524) (layers F.Cu F.Paste F.Mask)
+      (net 31 "Net-(IC1-Pad24)"))
+  )
   (gr_text "PS: Unlabled 0805 can be 0.1uF or nothing" (at 136 155 90) (layer F.SilkS)
     (effects (font (size 1.3 1) (thickness 0.25)))
@@
   (segment (start 204.75 159.5) (end 210.52 153.73) (width 1) (layer F.Cu) (net 25))
   (segment (start 118.235 152.985) (end 118.5 153.25) (width 0.25) (layer F.Cu) (net 25))
+  (segment (start 32.8 43.4) (end 30.65 43.4) (width 0.25) (layer F.Cu) (net 30))
+  (segment (start 30.65 43.4) (end 30.25 43) (width 0.25) (layer F.Cu) (net 30))
+  (segment (start 30.25 43) (end 30.25 42.5) (width 0.25) (layer F.Cu) (net 30))
+  (segment (start 30.25 42.5) (end 32.75 40) (width 0.25) (layer F.Cu) (net 30))
   (via (at 32.75 40) (size 0.6) (drill 0.4) (layers F.Cu B.Cu) (net 30))
   (segment (start 32.75 40) (end 32.8 40.05) (width 0.25) (layer F.Cu) (net 30))
-  (segment (start 32.8 40.05) (end 32.8 43.4) (width 0.25) (layer F.Cu) (net 30))
   (segment (start 124.25 162) (end 125.5 162) (width 0.25) (layer F.Cu) (net 30))
   (segment (start 125.5 162) (end 126.75 160.75) (width 0.25) (layer F.Cu) (net 30))
@@
   (segment (start 122 39.25) (end 33.5 39.25) (width 0.25) (layer B.Cu) (net 30))
   (segment (start 33.5 39.25) (end 32.75 40) (width 0.25) (layer B.Cu) (net 30))
-  (segment (start 36 40.5) (end 35.5 40.5) (width 0.25) (layer B.Cu) (net 31))
-  (segment (start 35.5 40.5) (end 34.5 41.5) (width 0.25) (layer B.Cu) (net 31))
-  (segment (start 34.5 41.5) (end 29.25 41.5) (width 0.25) (layer B.Cu) (net 31))
-  (segment (start 29.25 41.5) (end 27.75 43) (width 0.25) (layer B.Cu) (net 31))
-  (segment (start 27.75 43) (end 27.75 45) (width 0.25) (layer B.Cu) (net 31))
-  (via (at 27.75 45) (size 0.6) (drill 0.4) (layers F.Cu B.Cu) (net 31))
-  (segment (start 27.75 45) (end 32.8 45) (width 0.25) (layer F.Cu) (net 31))
-  (segment (start 122 40.5) (end 36 40.5) (width 0.25) (layer B.Cu) (net 31))
-  (segment (start 126 44.5) (end 122 40.5) (width 0.25) (layer B.Cu) (net 31))
-  (segment (start 126 71) (end 126 44.5) (width 0.25) (layer B.Cu) (net 31))
-  (segment (start 126 127.5) (end 126 71) (width 0.25) (layer B.Cu) (net 31))
-  (segment (start 126 156) (end 126 127.5) (width 0.25) (layer B.Cu) (net 31))
-  (segment (start 126 157) (end 126 156) (width 0.25) (layer B.Cu) (net 31))
-  (via (at 126 157) (size 0.6) (drill 0.4) (layers F.Cu B.Cu) (net 31))
-  (segment (start 126 160.5) (end 126 157) (width 0.25) (layer F.Cu) (net 31))
+  (segment (start 30.25 45.25) (end 32.55 45.25) (width 0.25) (layer F.Cu) (net 31))
+  (segment (start 32.55 45.25) (end 32.8 45) (width 0.25) (layer F.Cu) (net 31))
+  (segment (start 30.25 45.25) (end 28 45.25) (width 0.25) (layer F.Cu) (net 31))
+  (segment (start 125.3 161.2) (end 124.25 161.2) (width 0.25) (layer F.Cu) (net 31))
   (segment (start 125.3 161.2) (end 126 160.5) (width 0.25) (layer F.Cu) (net 31))
-  (segment (start 124.25 161.2) (end 125.3 161.2) (width 0.25) (layer F.Cu) (net 31))
+  (segment (start 126 160.5) (end 126 157) (width 0.25) (layer F.Cu) (net 31))
+  (via (at 126 157) (size 0.6) (drill 0.4) (layers F.Cu B.Cu) (net 31))
+  (segment (start 126 157) (end 126 156) (width 0.25) (layer B.Cu) (net 31))
+  (segment (start 126 156) (end 126 127.5) (width 0.25) (layer B.Cu) (net 31))
+  (segment (start 126 127.5) (end 126 71) (width 0.25) (layer B.Cu) (net 31))
+  (segment (start 126 71) (end 126 44.5) (width 0.25) (layer B.Cu) (net 31))
+  (segment (start 126 44.5) (end 122 40.5) (width 0.25) (layer B.Cu) (net 31))
+  (segment (start 122 40.5) (end 36 40.5) (width 0.25) (layer B.Cu) (net 31))
+  (via (at 27.75 45) (size 0.6) (drill 0.4) (layers F.Cu B.Cu) (net 31))
+  (segment (start 27.75 43) (end 27.75 45) (width 0.25) (layer B.Cu) (net 31))
+  (segment (start 29.25 41.5) (end 27.75 43) (width 0.25) (layer B.Cu) (net 31))
+  (segment (start 34.5 41.5) (end 29.25 41.5) (width 0.25) (layer B.Cu) (net 31))
+  (segment (start 35.5 40.5) (end 34.5 41.5) (width 0.25) (layer B.Cu) (net 31))
+  (segment (start 36 40.5) (end 35.5 40.5) (width 0.25) (layer B.Cu) (net 31))
+  (segment (start 28 45.25) (end 27.75 45) (width 0.25) (layer F.Cu) (net 31))
   (segment (start 124.25 161.2) (end 124.8 161.2) (width 0.6) (layer F.Cu) (net 31))
   (segment (start 61 49) (end 57 45) (width 0.25) (layer F.Cu) (net 34))
@@
   (segment (start 123.4 277.4) (end 127.8 277.4) (width 0.25) (layer F.Cu) (net 147))
   (segment (start 115.2 273.4) (end 119.4 273.4) (width 0.25) (layer F.Cu) (net 147))
-  (segment (start 291.54 270.25) (end 291.54 282.25) (width 0.25) (layer F.Cu) (net 148) (status 400000))
+  (segment (start 291.54 270.25) (end 291.54 282.25) (width 0.25) (layer F.Cu) (net 148))
   (segment (start 294.5 289) (end 293.2 289) (width 0.25) (layer F.Cu) (net 148))
   (segment (start 294.5 289) (end 295 288.5) (width 0.25) (layer F.Cu) (net 148))
@@
   (segment (start 291.54 282.79) (end 295 286.25) (width 0.25) (layer F.Cu) (net 148))
   (segment (start 291.54 282.25) (end 291.54 282.79) (width 0.25) (layer F.Cu) (net 148))
-  (segment (start 291.54 270.25) (end 292.04 269.75) (width 0.25) (layer F.Cu) (net 148) (status C00000))
-  (segment (start 289 270.25) (end 289 282.25) (width 0.25) (layer F.Cu) (net 149) (status 400000))
+  (segment (start 291.54 270.25) (end 292.04 269.75) (width 0.25) (layer F.Cu) (net 148))
+  (segment (start 289 270.25) (end 289 282.25) (width 0.25) (layer F.Cu) (net 149))
   (segment (start 289 283.375) (end 289 282.25) (width 0.25) (layer F.Cu) (net 149))
   (segment (start 289 283.375) (end 293.025 287.4) (width 0.25) (layer F.Cu) (net 149))
-  (segment (start 289 270.25) (end 289.5 269.75) (width 0.25) (layer F.Cu) (net 149) (status C00000))
+  (segment (start 289 270.25) (end 289.5 269.75) (width 0.25) (layer F.Cu) (net 149))
   (segment (start 293.2 287.4) (end 293.025 287.4) (width 0.25) (layer F.Cu) (net 149))
   (segment (start 257.8 49) (end 202.2 49) (width 0.25) (layer F.Cu) (net 150))
